Commit message: camera addition

File: description/robot.urdf.xacro (robot description, xacro)
@@ -3,3 +3,5 @@
     <xacro:include filename="robot_core.xacro" />
     <xacro:include filename="gazebo_control.xacro"/>
+    <xacro:include filename="lidar.xacro"/>
+    <xacro:include filename="camera.xacro"/>
 </robot>

File: description/robot_core.xacro (robot description, xacro)
@@ -11,7 +11,10 @@
         <color rgba="0.2 0.2 1 1"/>
     </material>
-    <material name="black">
-        <color rgba="0 0 0 1"/>
-    </material>
+        <material name="black">
+            <color rgba="0 0 0 1"/>
+        </material>
+        <material name="red">
+            <color rgba="1 0 0 1"/>
+        </material>
     <!--BASE LINK -->
     <link name="base_link">
